File: eagle/Chip/chip.brd (EAGLE design)
At the start: 160 x 100 mm, 58 parts, among them IC1 MCP604SL, J1 3x4 Keypad, Q2 BT137-600E, U1 328P, U2 TRIAC_OPTOCOUPLER-MOC3063SM, U3 SFH6206, Y1 16MHz

Commit message: added speaker to eagle
Parts:
- removed H1, H2, H3, H4, H5, H6, H7, H8, H9: STAND-OFF, SparkFun-Hardware:STAND-OFF
- removed T1: (no value), transistor-neu-to92:SOT23-BEC
- added J2: (no value), SparkFun-Connectors:1X02
- added LED1, LED2: (no value), adafruit:LED5MM
- added Q3, Q4: (no value), SparkFun-DiscreteSemi:SOT23-3
- added R18, R21: 150, adafruit:R0603
- added R19, R20: 2k, adafruit:R0603
Connections:
- new net N$38: LED1.K, Q3.3
- new net N$39: LED1.A, R18.1
- new net N$40: Q3.1, Q4.1, R19.2
- new net N$41: PIN_OUT.1, R20.1
- new net N$42: J2.2, Q4.3
- new net N$43: R19.1
- new net N$44: U1.28
- new net N$45: LED2.A, R21.1
- net 5V: now also J2.1, R18.2, R21.2
- net GND: now also LED2.K, Q3.2, Q4.2
- net N$35: now also R20.2; no longer PIN_OUT.1
Changed lines of the file:
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@@
 <attribute name="PROD_ID" value="CAP-00810" x="-64.77" y="91.44" size="1.778" layer="27" display="off"/>
 </element>
-<element name="H1" library="SparkFun-Hardware" library_urn="urn:adsk.eagle:library:519" package="STAND-OFF" package3d_urn="urn:adsk.eagle:package:38630/1" value="STAND-OFF" x="-78.74" y="74.93"/>
 <element name="H10" library="SparkFun-Hardware" library_urn="urn:adsk.eagle:library:519" package="STAND-OFF" package3d_urn="urn:adsk.eagle:package:38630/1" value="STAND-OFF" x="-60.96" y="86.36"/>
 <element name="H11" library="SparkFun-Hardware" library_urn="urn:adsk.eagle:library:519" package="STAND-OFF" package3d_urn="urn:adsk.eagle:package:38630/1" value="STAND-OFF" x="-67.31" y="86.36"/>
-<element name="H2" library="SparkFun-Hardware" library_urn="urn:adsk.eagle:library:519" package="STAND-OFF" package3d_urn="urn:adsk.eagle:package:38630/1" value="STAND-OFF" x="-85.09" y="74.93"/>
-<element name="H3" library="SparkFun-Hardware" library_urn="urn:adsk.eagle:library:519" package="STAND-OFF" package3d_urn="urn:adsk.eagle:package:38630/1" value="STAND-OFF" x="-16.51" y="86.36"/>
-<element name="H4" library="SparkFun-Hardware" library_urn="urn:adsk.eagle:library:519" package="STAND-OFF" package3d_urn="urn:adsk.eagle:package:38630/1" value="STAND-OFF" x="-22.86" y="86.36"/>
-<element name="H5" library="SparkFun-Hardware" library_urn="urn:adsk.eagle:library:519" package="STAND-OFF" package3d_urn="urn:adsk.eagle:package:38630/1" value="STAND-OFF" x="-29.21" y="86.36"/>
-<element name="H6" library="SparkFun-Hardware" library_urn="urn:adsk.eagle:library:519" package="STAND-OFF" package3d_urn="urn:adsk.eagle:package:38630/1" value="STAND-OFF" x="-35.56" y="86.36"/>
-<element name="H7" library="SparkFun-Hardware" library_urn="urn:adsk.eagle:library:519" package="STAND-OFF" package3d_urn="urn:adsk.eagle:package:38630/1" value="STAND-OFF" x="-41.91" y="86.36"/>
-<element name="H8" library="SparkFun-Hardware" library_urn="urn:adsk.eagle:library:519" package="STAND-OFF" package3d_urn="urn:adsk.eagle:package:38630/1" value="STAND-OFF" x="-48.26" y="86.36"/>
-<element name="H9" library="SparkFun-Hardware" library_urn="urn:adsk.eagle:library:519" package="STAND-OFF" package3d_urn="urn:adsk.eagle:package:38630/1" value="STAND-OFF" x="-54.61" y="86.36"/>
 <element name="J1" library="SparkFun-Connectors" library_urn="urn:adsk.eagle:library:513" package="1X07" package3d_urn="urn:adsk.eagle:package:38129/1" value="3x4 Keypad" x="-30.48" y="92.71"/>
 <element name="L1" library="SparkFun-Coils" library_urn="urn:adsk.eagle:library:512" package="0603" package3d_urn="urn:adsk.eagle:package:37574/1" value="10uH" x="-83.82" y="91.44">
@@
 </element>
 <element name="R3" library="resistor" library_urn="urn:adsk.eagle:library:348" package="RTRIM3296W" package3d_urn="urn:adsk.eagle:package:26033/1" value="10k" x="-45.72" y="45.72"/>
-<element name="T1" library="transistor-neu-to92" library_urn="urn:adsk.eagle:library:397" package="SOT23-BEC" package3d_urn="urn:adsk.eagle:package:28748/2" value="" x="-72.39" y="85.09"/>
 <element name="U1" library="SparkFun-IC-Microcontroller" library_urn="urn:adsk.eagle:library:525" package="DIP28" package3d_urn="urn:adsk.eagle:package:38942/1" value="328P" x="-33.02" y="77.47">
 <attribute name="PROD_ID" value="IC-09136" x="-33.02" y="77.47" size="1.778" layer="27" display="off"/>
@@
 <element name="PIN_IN" library="SparkFun-Connectors" library_urn="urn:adsk.eagle:library:513" package="1X01" package3d_urn="urn:adsk.eagle:package:38028/1" value="" x="-85.3186" y="-76.5048"/>
 <element name="PIN_OUT" library="SparkFun-Connectors" library_urn="urn:adsk.eagle:library:513" package="1X01" package3d_urn="urn:adsk.eagle:package:38028/1" value="" x="-85.3186" y="-95.3008"/>
+<element name="LED1" library="adafruit" library_urn="urn:adsk.eagle:library:420" package="LED5MM" value="" x="-85.0646" y="-132.8674"/>
+<element name="R18" library="adafruit" library_urn="urn:adsk.eagle:library:420" package="R0603" value="150" x="-93.218" y="-143.9672"/>
+<element name="Q3" library="SparkFun-DiscreteSemi" library_urn="urn:adsk.eagle:library:514" package="SOT23-3" package3d_urn="urn:adsk.eagle:package:38446/1" value="" x="-97.2058" y="-143.9926">
+<attribute name="PROD_ID" value="TRANS-09116" x="-97.2058" y="-143.9926" size="1.778" layer="27" display="off"/>
+</element>
+<element name="R19" library="adafruit" library_urn="urn:adsk.eagle:library:420" package="R0603" value="2k" x="-98.2472" y="-149.225"/>
+<element name="Q4" library="SparkFun-DiscreteSemi" library_urn="urn:adsk.eagle:library:514" package="SOT23-3" package3d_urn="urn:adsk.eagle:package:38446/1" value="" x="-102.235" y="-149.2504">
+<attribute name="PROD_ID" value="TRANS-09116" x="-102.235" y="-149.2504" size="1.778" layer="27" display="off"/>
+</element>
+<element name="R20" library="adafruit" library_urn="urn:adsk.eagle:library:420" package="R0603" value="2k" x="-103.2764" y="-154.4828"/>
+<element name="J2" library="SparkFun-Connectors" library_urn="urn:adsk.eagle:library:513" package="1X02" package3d_urn="urn:adsk.eagle:package:38039/1" value="" x="-95.377" y="-166.4208"/>
+<element name="R21" library="adafruit" library_urn="urn:adsk.eagle:library:420" package="R0603" value="150" x="-103.2764" y="-178.5366"/>
+<element name="LED2" library="adafruit" library_urn="urn:adsk.eagle:library:420" package="LED5MM" value="" x="-95.123" y="-189.4586"/>
 </elements>
 <signals>
@@
 <contactref element="U3" pad="3"/>
 <contactref element="Q1" pad="2"/>
+<contactref element="Q3" pad="2"/>
+<contactref element="Q4" pad="2"/>
+<contactref element="LED2" pad="K"/>
+<wire x1="-96.2558" y1="-144.9926" x2="-101.285" y2="-150.2504" width="0" layer="19" extent="1-1"/>
+<wire x1="-82.8954" y1="-122.8184" x2="-96.2558" y2="-144.9926" width="0" layer="19" extent="1-1"/>
 <wire x1="-70.2818" y1="-89.2608" x2="-82.8954" y2="-122.8184" width="0" layer="19" extent="1-1"/>
+<wire x1="-93.853" y1="-189.4586" x2="-101.285" y2="-150.2504" width="0" layer="19" extent="1-1"/>
 <wire x1="-75.18" y1="35.82" x2="-70.2818" y2="-89.2608" width="0" layer="19" extent="1-1"/>
 <wire x1="-85.34" y1="35.82" x2="-75.18" y2="35.82" width="0" layer="19" extent="1-1"/>
@@
 <contactref element="R15" pad="1"/>
 <contactref element="R16" pad="2"/>
+<contactref element="R18" pad="2"/>
+<contactref element="J2" pad="1"/>
+<contactref element="R21" pad="2"/>
+<wire x1="-94.068" y1="-121.9454" x2="-92.368" y2="-143.9672" width="0" layer="19" extent="1-1"/>
+<wire x1="-95.377" y1="-166.4208" x2="-92.368" y2="-143.9672" width="0" layer="19" extent="1-1"/>
+<wire x1="-102.4264" y1="-178.5366" x2="-95.377" y2="-166.4208" width="0" layer="19" extent="1-1"/>
 <wire x1="-70.1684" y1="-107.4166" x2="-94.068" y2="-121.9454" width="0" layer="19" extent="1-1"/>
 <wire x1="-70.3462" y1="-41.5798" x2="-70.1684" y2="-107.4166" width="0" layer="19" extent="1-1"/>
@@
 <wire x1="-83.8454" y1="-120.7184" x2="-89.6366" y2="-116.4082" width="0" layer="19" extent="1-1"/>
 </signal>
-<signal name="N$35">
-<contactref element="Q1" pad="1"/>
-<contactref element="PIN_OUT" pad="1"/>
-<wire x1="-85.3186" y1="-95.3008" x2="-84.7954" y2="-122.8184" width="0" layer="19" extent="1-1"/>
-</signal>
 <signal name="N$36">
 <contactref element="Q2" pad="2"/>
@@
 <wire x1="-80.8482" y1="-112.1156" x2="-81.6728" y2="-121.9454" width="0" layer="19" extent="1-1"/>
 </signal>
+<signal name="N$39">
+<contactref element="LED1" pad="A"/>
+<contactref element="R18" pad="1"/>
+<wire x1="-86.3346" y1="-132.8674" x2="-94.068" y2="-143.9672" width="0" layer="19" extent="1-1"/>
+</signal>
+<signal name="N$38">
+<contactref element="LED1" pad="K"/>
+<contactref element="Q3" pad="3"/>
+<wire x1="-83.7946" y1="-132.8674" x2="-97.2058" y2="-142.8926" width="0" layer="19" extent="1-1"/>
+</signal>
+<signal name="N$40">
+<contactref element="Q3" pad="1"/>
+<contactref element="R19" pad="2"/>
+<contactref element="Q4" pad="1"/>
+<wire x1="-97.3972" y1="-149.225" x2="-103.185" y2="-150.2504" width="0" layer="19" extent="1-1"/>
+<wire x1="-98.1558" y1="-144.9926" x2="-97.3972" y2="-149.225" width="0" layer="19" extent="1-1"/>
+</signal>
+<signal name="N$35">
+<contactref element="Q1" pad="1"/>
+<contactref element="R20" pad="2"/>
+<wire x1="-102.4264" y1="-154.4828" x2="-84.7954" y2="-122.8184" width="0" layer="19" extent="1-1"/>
+</signal>
+<signal name="N$41">
+<contactref element="PIN_OUT" pad="1"/>
+<contactref element="R20" pad="1"/>
+<wire x1="-104.1264" y1="-154.4828" x2="-85.3186" y2="-95.3008" width="0" layer="19" extent="1-1"/>
+</signal>
+<signal name="N$42">
+<contactref element="Q4" pad="3"/>
+<contactref element="J2" pad="2"/>
+<wire x1="-92.837" y1="-166.4208" x2="-102.235" y2="-148.1504" width="0" layer="19" extent="1-1"/>
+</signal>
+<signal name="N$43">
+<contactref element="R19" pad="1"/>
+</signal>
+<signal name="N$44">
+<contactref element="U1" pad="28"/>
+</signal>
+<signal name="N$45">
+<contactref element="R21" pad="1"/>
+<contactref element="LED2" pad="A"/>
+<wire x1="-104.1264" y1="-178.5366" x2="-96.393" y2="-189.4586" width="0" layer="19" extent="1-1"/>
+</signal>
 </signals>
