File: eagle/Chip/Granny Safe all Inclusive.sch (EAGLE design)
At the start: 52 parts, among them IC1 MCP604SL, J1 3x4 Keypad, J3 SCREW-4, J4 i2c_16x2, J6 FEMALE 2x3, Q1 TRANS_NPN-MMBTA42, Q2 TRANS_NPN-MMBTA42, Q3 TRANS_NPN-MMBTA42, U1 328P

Commit message: Put both schematics together
Parts:
- added C10: 100pF, SparkFun-Capacitors:100PF-0603-50V-5%
- added C11: 1nF, SparkFun-Capacitors:1.0NF/1000PF-0603-50V-10%
- added C3, C7: 470u, adafruit:CPOL-USE3.5-8
- added C8: 100u, adafruit:CPOL-USE2-5
- added C9: 0.1uF, SparkFun-Capacitors:0.1UF-0603-25V-5%
- added D1, D2, D3, D4, D5: DIODE-SCHOTTKY-B340A, SparkFun-DiscreteSemi:DIODE-SCHOTTKY-B340A
- added F1: 1.5A, fuse:TE5
- added IC2: LM2596S, national-semiconductor:LM2596S
- added J10: AC GND CONN, SparkFun-Connectors:CONN_025MM
- added J7: (no value), SparkFun-Connectors:CONN_04
- added J8: 120V Plug, SparkFun-Connectors:CONN_025MM
- added J9: Hotplate Outlet, SparkFun-Connectors:CONN_025MM
- added L2: INDUCTOR, ece:INDUCTOR
- added Q4: 2N3904, SparkFun-DiscreteSemi:TRANS_NPN-MMBTA42
- added R20, R23: 10k, adafruit:R-US_R0603
- added R22: 220, adafruit:R-US_R0603
- added R24: 180, adafruit:R-US_R0603
- added R25: 2k, adafruit:R-US_R0603
- added R26: 3.3k, SparkFun-Resistors:3.3KOHM-0603-1/10W-1%
- added R27: 1k, SparkFun-Resistors:1KOHM-0603-1/10W-1%
- added T1: BT137, ece:BT137
- added U2: SFH6206, optocoupler:SFH6206
- added U3: MOC3051, ece:MOC3051
- added VR2: 10k, SparkFun-Resistors:TRIMPOT-SMD-3MM-OPEN-1/10W-25%
- added XFMR1: EE20-2, ece:EE20-2
Connections:
- new net +5V: J7.3, R22.1
- new net AC_GND: J10.1, J10.2
- new net LINE: J8.1, T1.A2, U3.6, XFMR1.2
- new net N$22: D2.C, D3.A, F1.2
- new net N$29: R20.2, U2.AC1
- new net N$30: R24.2, T1.G
- new net N$31: R22.2, U3.1
- new net N$32: R24.1, U3.4
- new net N$33: IC2.FB, R26.1, R27.2, VR2.WIPER
- new net N$34: Q4.C, U3.2
- new net N$35: Q4.B, R25.2
- new net N$36: C10.1, C11.1, C7.+, C9.1, L2.2, R26.2, VR2.CW
- new net N$37: F1.1, XFMR1.4, XFMR1.6
- new net N$41: D4.A, D5.A, XFMR1.3, XFMR1.5
- new net N$46: D1.C, IC2.OUT, L2.1
- new net N$51: C3.+, C8.+, D3.C, D5.C, IC2.VIN
- new net NEUT: J8.2, J9.2, XFMR1.1
- new net PWR: J9.1, T1.A1
- new net ZS: R23.1, U2.C
- net 5V: now also R23.2, TP4.1
- net ALR: now also TP7.1
- net GATE: now also J7.1, R25.1
- net GND: now also C10.2, C11.2, C3.-, C7.-, C8.-, C9.2, D1.A, D2.A, D4.C, IC2.!ON!/OFF, IC2.GND, Q4.E, R27.1, TP3.1, U2.E, VR2.CCW
- net SET: now also TP5.1
- net T_EN: now also TP6.1
Other:
- note added: "25V"
- note added: "330u"
- note added: "LM2576"
- note added: "U3"
- moved on the sheet: C1, C2, C4, C5, C6, IC1A, IC1B, IC1C, IC1D, J1, J2, J3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
