File: eagle/Chip/Granny Safe.sch (EAGLE design)
At the start: 87 parts, among them IC1 MCP604SL, IC2 LM2596S, J1 3x4 Keypad, J10 SCREW-4, J2 FEMALE 2x3, J3 SCREW-4, J4 i2c_16x2, J6 FEMALE 2x3, J8 RES JUMPER, J9 CKT PWR CONN, Q1 TRANS_NPN-MMBTA42, Q2 TRANS_NPN-MMBTA42, Q3 TRANS_NPN-MMBTA42, Q4 2N3904, T1 BT137, U1 328P, U2 SFH6206, U3 MOC3051

Commit message: Updated board
Parts:
- renumbered LED1 to ALR_LED, LED3 to SET_LED, LED4 to TIM_LED, LED5 to ON_LED
Changed lines of the file:
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@@
 <part name="RTD" library="SparkFun-Resistors" library_urn="urn:adsk.eagle:library:532" deviceset="10KOHM" device="-HORIZ-1/4W-1%" package3d_urn="urn:adsk.eagle:package:39658/1" value=""/>
 <part name="SUPPLY8" library="SparkFun-PowerSymbols" library_urn="urn:adsk.eagle:library:530" deviceset="5V" device=""/>
-<part name="LED1" library="adafruit" library_urn="urn:adsk.eagle:library:420" deviceset="LED" device="5MM"/>
+<part name="ALR_LED" library="adafruit" library_urn="urn:adsk.eagle:library:420" deviceset="LED" device="5MM"/>
 <part name="R18" library="adafruit" library_urn="urn:adsk.eagle:library:420" deviceset="R-US_" device="R0603" value="150"/>
 <part name="Q3" library="SparkFun-DiscreteSemi" library_urn="urn:adsk.eagle:library:514" deviceset="TRANS_NPN" device="-MMBTA42" package3d_urn="urn:adsk.eagle:package:38446/1" value=""/>
@@
 <part name="R14" library="adafruit" library_urn="urn:adsk.eagle:library:420" deviceset="R-US_" device="R0603" value="150"/>
 <part name="R15" library="adafruit" library_urn="urn:adsk.eagle:library:420" deviceset="R-US_" device="R0603" value="150"/>
-<part name="LED3" library="adafruit" library_urn="urn:adsk.eagle:library:420" deviceset="LED" device="5MM"/>
-<part name="LED4" library="adafruit" library_urn="urn:adsk.eagle:library:420" deviceset="LED" device="5MM"/>
+<part name="SET_LED" library="adafruit" library_urn="urn:adsk.eagle:library:420" deviceset="LED" device="5MM"/>
+<part name="TIM_LED" library="adafruit" library_urn="urn:adsk.eagle:library:420" deviceset="LED" device="5MM"/>
 <part name="SUPPLY4" library="SparkFun-PowerSymbols" library_urn="urn:adsk.eagle:library:530" deviceset="5V" device=""/>
 <part name="SUPPLY9" library="SparkFun-PowerSymbols" library_urn="urn:adsk.eagle:library:530" deviceset="5V" device=""/>
@@
 <part name="GND11" library="SparkFun-PowerSymbols" deviceset="GND" device=""/>
 <part name="R28" library="adafruit" library_urn="urn:adsk.eagle:library:420" deviceset="R-US_" device="R0603" value="150"/>
-<part name="LED5" library="adafruit" library_urn="urn:adsk.eagle:library:420" deviceset="LED" device="5MM"/>
+<part name="ON_LED" library="adafruit" library_urn="urn:adsk.eagle:library:420" deviceset="LED" device="5MM"/>
 <part name="GND12" library="SparkFun-PowerSymbols" deviceset="GND" device=""/>
 <part name="SUPPLY13" library="SparkFun-PowerSymbols" library_urn="urn:adsk.eagle:library:530" deviceset="5V" device=""/>
@@
 <instance part="RTD" gate="G$1" x="12.7" y="165.1" rot="MR0"/>
 <instance part="SUPPLY8" gate="G$1" x="86.36" y="167.64"/>
-<instance part="LED1" gate="G$1" x="109.22" y="25.4" smashed="yes">
+<instance part="ALR_LED" gate="G$1" x="109.22" y="25.4" smashed="yes">
 <attribute name="NAME" x="106.172" y="26.416" size="1.778" layer="95" rot="R180"/>
 <attribute name="VALUE" x="114.935" y="20.828" size="1.778" layer="96" rot="R90"/>
@@
 <attribute name="VALUE" x="26.67" y="33.782" size="1.778" layer="96" rot="R180"/>
 </instance>
-<instance part="LED3" gate="G$1" x="30.48" y="25.4" smashed="yes">
+<instance part="SET_LED" gate="G$1" x="30.48" y="25.4" smashed="yes">
 <attribute name="NAME" x="27.432" y="26.416" size="1.778" layer="95" rot="R180"/>
 <attribute name="VALUE" x="36.195" y="20.828" size="1.778" layer="96" rot="R90"/>
 </instance>
-<instance part="LED4" gate="G$1" x="66.04" y="25.4" smashed="yes">
+<instance part="TIM_LED" gate="G$1" x="66.04" y="25.4" smashed="yes">
 <attribute name="NAME" x="62.992" y="26.416" size="1.778" layer="95" rot="R180"/>
 <attribute name="VALUE" x="71.755" y="20.828" size="1.778" layer="96" rot="R90"/>
@@
 <attribute name="VALUE" x="223.52" y="63.246" size="1.778" layer="96" rot="R180"/>
 </instance>
-<instance part="LED5" gate="G$1" x="218.186" y="55.626" smashed="yes">
-<attribute name="NAME" x="225.806" y="55.118" size="1.778" layer="95" rot="R180"/>
+<instance part="ON_LED" gate="G$1" x="218.186" y="55.626" smashed="yes">
+<attribute name="NAME" x="229.108" y="55.118" size="1.778" layer="95" rot="R180"/>
 <attribute name="VALUE" x="223.901" y="51.054" size="1.778" layer="96" rot="R90"/>
 </instance>
@@
 </segment>
 <segment>
-<pinref part="LED5" gate="G$1" pin="C"/>
+<pinref part="ON_LED" gate="G$1" pin="C"/>
 <pinref part="GND12" gate="1" pin="GND"/>
 <pinref part="J12" gate="G$1" pin="2"/>
@@
 <net name="N$39" class="0">
 <segment>
-<pinref part="LED1" gate="G$1" pin="A"/>
+<pinref part="ALR_LED" gate="G$1" pin="A"/>
 <pinref part="R18" gate="G$1" pin="1"/>
 <wire x1="109.22" y1="27.94" x2="115.316" y2="27.94" width="0.1524" layer="91"/>
@@
 <segment>
 <pinref part="R15" gate="G$1" pin="1"/>
-<pinref part="LED3" gate="G$1" pin="A"/>
+<pinref part="SET_LED" gate="G$1" pin="A"/>
 <pinref part="J7" gate="G$1" pin="1"/>
 <wire x1="35.56" y1="25.4" x2="35.56" y2="27.94" width="0.1524" layer="91"/>
@@
 <segment>
 <pinref part="R14" gate="G$1" pin="1"/>
-<pinref part="LED4" gate="G$1" pin="A"/>
+<pinref part="TIM_LED" gate="G$1" pin="A"/>
 <pinref part="J11" gate="G$1" pin="1"/>
 <wire x1="71.12" y1="25.4" x2="71.12" y2="27.94" width="0.1524" layer="91"/>
@@
 <net name="N$19" class="0">
 <segment>
-<pinref part="LED4" gate="G$1" pin="C"/>
+<pinref part="TIM_LED" gate="G$1" pin="C"/>
 <pinref part="Q2" gate="G$1" pin="C"/>
 <pinref part="J11" gate="G$1" pin="2"/>
@@
 <net name="N$20" class="0">
 <segment>
-<pinref part="LED3" gate="G$1" pin="C"/>
+<pinref part="SET_LED" gate="G$1" pin="C"/>
 <pinref part="Q1" gate="G$1" pin="C"/>
 <wire x1="30.48" y1="20.32" x2="35.56" y2="20.32" width="0.1524" layer="91"/>
@@
 <net name="N$23" class="0">
 <segment>
-<pinref part="LED1" gate="G$1" pin="C"/>
+<pinref part="ALR_LED" gate="G$1" pin="C"/>
 <pinref part="Q3" gate="G$1" pin="C"/>
 <wire x1="109.22" y1="20.32" x2="115.316" y2="20.32" width="0.1524" layer="91"/>
@@
 <segment>
 <pinref part="R28" gate="G$1" pin="1"/>
-<pinref part="LED5" gate="G$1" pin="A"/>
+<pinref part="ON_LED" gate="G$1" pin="A"/>
 <pinref part="J12" gate="G$1" pin="1"/>
 <wire x1="231.648" y1="55.626" x2="231.648" y2="58.166" width="0.1524" layer="91"/>
