File: eagle/Chip/Granny Safe.brd (EAGLE design)
At the start: 160 x 100 mm, 87 parts, among them IC1 MCP604SL, IC2 LM2596S, J1 3x4 Keypad, J10 SCREW-4, J2 FEMALE 2x3, J3 SCREW-4, J4 i2c_16x2, J6 FEMALE 2x3, J8 RES JUMPER, J9 CKT PWR CONN, Q4 2N3904, T1 BT137, U1 328P, U2 SFH6206, U3 MOC3051

Commit message: Updated board
Parts:
- removed LED1, LED3, LED4, LED5: (no value), adafruit:LED5MM
- added ALR_LED, ON_LED, SET_LED, TIM_LED: (no value), adafruit:LED5MM
- moved R16 224.5 mm to (123.2, 20.3), turned to 90 degrees
- moved Q4 214.1 mm to (123.2, 31.8), turned to 270 degrees
- moved R19 211.9 mm to (102.9, 16.5), turned to 180 degrees
- moved R18 211.3 mm to (102.9, 7.62), turned to 270 degrees
- moved XTAL 200.7 mm to (106.7, 58.4), turned to 270 degrees
- moved R8 200.2 mm to (85.1, 40.6)
- moved J2 197.3 mm to (106.7, 17.8), turned to 270 degrees
- moved R15 196.9 mm to (91.4, 7.62), turned to 270 degrees
- moved C2 192.4 mm to (102.9, 61.0), turned to 270 degrees
- moved C1 190.6 mm to (102.9, 55.9), turned to 90 degrees
- moved R6 188.7 mm to (83.8, 43.2), turned to 180 degrees
- moved C5 187.5 mm to (87.6, 54.6), turned to 180 degrees
- moved Q3 185.1 mm to (102.9, 12.7), turned to 270 degrees
- moved R7 184.6 mm to (69.8, 33.0)
- moved R14 182.8 mm to (80.0, 7.62), turned to 270 degrees
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Connections:
- net GND: now also ON_LED.K; no longer LED5.K
- net N$17: now also SET_LED.A; no longer LED3.A
- net N$18: now also TIM_LED.A; no longer LED4.A
- net N$19: now also TIM_LED.K; no longer LED4.K
- net N$20: now also SET_LED.K; no longer LED3.K
- net N$23: now also ALR_LED.K; no longer LED1.K
- net N$36: now also ON_LED.A; no longer LED5.A
- net N$39: now also ALR_LED.A; no longer LED1.A
Routing:
- net N$33: track 0.00 -> 11.1 mm, vias 0 -> 1
- net N$51: track 0.00 -> 5.08 mm
- net N$46: track 0.00 -> 4.55 mm
- net N$41: track 0.00 -> 3.32 mm
- net N$22: track 0.00 -> 3.32 mm
- added copper zone on layer 1, net GND
Other:
- board size 160 x 100 mm -> 99 x 100 mm

Commit message: worked on board some more
Parts:
- moved U2 29.6 mm to (111.8, 43.2), turned to 180 degrees
- moved IC1 26.2 mm to (83.8, 69.8)
- moved J10 23.9 mm to (144.8, 43.2), turned to 180 degrees
- moved U3 18.1 mm to (118.1, 43.2)
- moved T1 15.3 mm to (157.5, 43.2)
- moved R20 15.3 mm to (125.7, 21.6)
- moved C7 15.2 mm to (81.3, 95.2), turned to 90 degrees
- moved J11 14.0 mm to (85.1, 26.7)
- moved J12 14.0 mm to (71.1, 26.7)
- moved J7 14.0 mm to (96.5, 26.7)
- moved Q1 14.0 mm to (92.7, 26.7)
- moved Q2 14.0 mm to (80.0, 26.7)
- moved Q3 14.0 mm to (102.9, 26.7)
- moved ALR_LED 14.0 mm to (108.0, 21.6)
- moved J2 14.0 mm to (106.7, 31.8)
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Routing:
- net LINE: track 0.00 -> 63.5 mm, vias 0 -> 37
- net NEUT: track 0.00 -> 63.0 mm, vias 0 -> 16
- net PWR: track 0.00 -> 31.0 mm, vias 0 -> 11
- added copper zone on layer 1, net LINE
- added copper zone on layer 16, net LINE
- added copper zone on layer 1, net N$4
- added copper zone on layer 1, net NEUT
- added copper zone on layer 16, net NEUT
- added copper zone on layer 1, net PWR
- added copper zone on layer 16, net PWR
- removed copper zone on layer 1, net GND
Other:
- board size 99 x 100 mm -> 99 x 83 mm

Commit message: Worked on the board some more
Parts:
- moved H1 290.5 mm to (164.8, 98.6)
- moved H4 284.3 mm to (154.9, 35.1)
- moved H2 192.3 mm to (50.0, 98.6)
- moved H3 167.3 mm to (45.2, 20.3)
- moved R24 32.2 mm to (114.6, 54.1), turned to 90 degrees
- moved R16 24.0 mm to (110.7, 40.9), turned to 270 degrees
- moved R23 21.8 mm to (109.2, 40.9)
- moved R25 20.6 mm to (104.4, 47.0), turned to 0 degrees
- moved Q4 20.4 mm to (110.0, 47.2)
- moved R20 16.1 mm to (123.7, 37.6)
- moved R22 15.4 mm to (112.5, 50.3)
- moved U2 6.51 mm to (117.9, 40.9), turned to 90 degrees
- moved U3 5.00 mm to (120.1, 47.8)
- moved J5 3.56 mm to (104.4, 36.8)
- moved TP1 3.56 mm to (104.4, 44.5)
Routing:
- net N$30: track 0.00 -> 68.2 mm
- net NEUT: track 63.0 -> 112.7 mm, vias 16 -> 17
- net N$32: track 0.00 -> 14.6 mm, vias 0 -> 2
- net LINE: track 63.5 -> 50.6 mm, vias 37 -> 26
- net ZERO: track 0.00 -> 4.11 mm
- net PWR: track 31.0 -> 27.2 mm, vias 11 -> 9
- net GND: track 0.00 -> 2.52 mm
- net N$29: track 0.00 -> 2.12 mm
- added copper zone on layer 1, net GND
- removed copper zone on layer 1, net N$4
