File: eagle/Chip/Granny Safe.brd (EAGLE design)
At the start: 113.5 x 64.8 mm, 87 parts, among them IC1 MCP604SL, IC2 LM2596S, J1 3x4 Keypad, J10 SCREW-4, J2 FEMALE 2x3, J3 SCREW-4, J4 i2c_16x2, J6 FEMALE 2x3, J8 RES JUMPER, J9 CKT PWR CONN, Q4 2N3904, T1 BT137, U1 328P, U2 SFH6206, U3 MOC3051

Commit message: worked on the board some more
should be pretty close to being done
Parts:
- removed IC2: LM2596S, national-semiconductor:TO263-5
- removed J9: CKT PWR CONN, SparkFun-Connectors:1X02
- removed TP4: (no value), SparkFun-Connectors:1X01
- added IC3: (no value), linear:TO263-5
- added S1: EG1213, adafruit:EG1213
- moved ON_LED 52.5 mm to (88.6, 71.9), turned to 180 degrees
- moved R18 49.8 mm to (64.3, 53.1), turned to 90 degrees
- moved ALR_LED 49.3 mm to (66.8, 48.8), turned to 270 degrees
- moved R28 48.5 mm to (85.6, 67.1), turned to 0 degrees
- moved J12 44.5 mm to (83.6, 69.3), turned to 90 degrees
- moved Q3 43.0 mm to (69.1, 53.3), turned to 180 degrees
- moved R1 39.1 mm to (98.0, 69.6), turned to 180 degrees
- moved J2 38.7 mm to (71.9, 48.8), turned to 0 degrees
- moved R19 38.4 mm to (72.6, 54.1)
- moved Q1 34.6 mm to (62.5, 43.4), turned to 180 degrees
- moved SET_LED 34.0 mm to (67.8, 39.9)
- moved XTAL 33.3 mm to (76.2, 68.3), turned to 0 degrees
- moved C2 32.6 mm to (73.7, 72.4)
- moved J7 31.3 mm to (70.4, 43.9), turned to 180 degrees
- moved J5 30.7 mm to (98.8, 67.1), turned to 180 degrees
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Connections:
- new net N$4: J8.1, S1.3
- net 5V: now also S1.1; no longer J9.2, TP4.1
- net GND: now also IC3.3, IC3.5, IC3.6; no longer IC2.3, IC2.5
- net N$33: now also IC3.4; no longer IC2.4
- net N$38: now also J8.3, S1.2; no longer J8.1, J9.1
- net N$46: now also IC3.2; no longer IC2.2
- net N$51: now also IC3.1; no longer IC2.1
Routing:
- net N$41: track 20.6 -> 53.5 mm
- net N$38: track 0.00 -> 30.9 mm, vias 0 -> 1
- net N$51: track 0.00 -> 30.0 mm
- net N$33: track 0.00 -> 29.0 mm, vias 0 -> 3
- net N$37: track 20.1 -> 40.7 mm
- net N$22: track 0.00 -> 18.9 mm
- net 5V: track 0.00 -> 14.9 mm
- net N$46: track 0.00 -> 13.0 mm
- net LINE: track 50.6 -> 59.3 mm
- net N$4: track 0.00 -> 8.25 mm
- net GND: track 2.52 -> 10.2 mm, vias 0 -> 36
- added copper zone on layer 16, net GND
Other:
- board size 113.5 x 64.8 mm -> 104.6 x 64.8 mm
